Commit message: added moveit

File: src/chessbot_description/urdf/arm_core.urdf.xacro (robot description, xacro)
@@ -17,4 +17,13 @@
   <xacro:property name="a3" default="0.115"/>
   <xacro:property name="a4" default="0.19"/>
+  <xacro:macro name="arm_default_transmission" params="joint_number" >
+      <plugin>transmission_interface/SimpleTransmission</plugin>
+      <transmission name="transmission_${joint_number}">
+          <joint name="joint${joint_number}" role="joint1">
+              <mechanicalReduction>1.0</mechanicalReduction>
+          </joint>
+          <actuator name="servo${joint_number}" role="actuator1"/>
+      </transmission>
+  </xacro:macro>
   <link name="base_link">
     <visual>
@@ -93,24 +102,232 @@
   <link name="arm1">
     <visual>
-      <origin xyz="0.0 0.0 0.0" rpy="0.0 0.0 0.0"/>
-      <geometry>
-        <box size="${a2} 0.04 0.001"/>
-      </geometry>
-      <material name="grey"/>
-    </visual>
-    <collision>
-      <origin xyz="0.0 0.0 0.0" rpy="0.0 0.0 0.0"/>
+      <origin xyz="${-a2/2} 0.0 0.0" rpy="0.0 0.0 0.0"/>
       <geometry>
         <box size="${a2} 0.02 0.001"/>
       </geometry>
       <material name="grey"/>
+    </visual>
+    <collision>
+      <origin xyz="${-a2/2} 0.0 0.0" rpy="0.0 0.0 0.0"/>
+      <geometry>
+        <box size="${a2} 0.02 0.001"/>
+      </geometry>
+      <material name="grey"/>
     </collision>
     <xacro:box mass="0.2" length="${a2}" width="0.001" height="0.02"
-          xyz="0.0 0.0 0.0" rpy="0.0 0.0 0.0"/>
+          xyz="${-a2/2} 0.0 0.0" rpy="0.0 0.0 0.0"/>
   </link>
   <joint name="arm_joint" type="fixed">
     <parent link="servo2"/>
     <child link="arm1"/>
-    <origin xyz="0.0 0.0 0.0" rpy="0.0 0.0 0.0"/>
-  </joint>
+    <origin xyz="${a2} 0.0 0.0" rpy="0.0 0.0 0.0"/>
+  </joint>
+  <link name="servo3">
+    <visual>
+      <origin xyz="0.0 0.0 ${servo_length/2}" rpy="0.0 0.0 0.0"/>
+      <geometry>
+        <cylinder radius="${servo_radius}" length="${servo_length}"/>
+      </geometry>
+      <material name="black"/>
+    </visual>
+    <collision>
+      <origin xyz="0.0 0.0 ${servo_length/2}" rpy="0.0 0.0 0.0"/>
+      <geometry>
+        <cylinder radius="${servo_radius}" length="${servo_length}"/>
+      </geometry>
+      <material name="black"/>
+    </collision>
+    <xacro:cylinder mass="2" radius="${servo_radius}" height="${servo_length}"
+            xyz="0.0 0.0 ${servo_length/2}" rpy="0.0 0.0 0.0"/>
+  </link>
+  <joint name="joint3" type="revolute">
+    <parent link="arm1"/>
+    <child link="servo3"/>
+    <axis xyz="0 0 1"/>
+    <limit lower="0" upper="${PI}" velocity="50.0" effort="1000.0"/>
+    <origin xyz="0 0 0" rpy="${PI} 0 0"/>
+  </joint>
+  <link name="servo4">
+    <visual>
+      <origin xyz="0.0 0.0 ${-0.103/2}" rpy="0.0 0.0 0.0"/>
+      <geometry>
+        <cylinder radius="${servo_radius}" length="0.103"/>
+      </geometry>
+      <material name="black"/>
+    </visual>
+    <collision>
+      <origin xyz="0.0 0.0 ${-0.103/2}" rpy="0.0 0.0 0.0"/>
+      <geometry>
+        <cylinder radius="${servo_radius}" length="0.103"/>
+      </geometry>
+      <material name="black"/>
+    </collision>
+    <xacro:cylinder mass="2" radius="${servo_radius}" height="${servo_length}"
+            xyz="0.0 0.0 ${-0.103/2}" rpy="0.0 0.0 0.0"/>
+  </link>
+  <joint name="joint4" type="revolute">
+    <parent link="servo3"/>
+    <child link="servo4"/>
+    <axis xyz="0 0 1"/>
+    <limit lower="0" upper="${PI}" velocity="50.0" effort="1000.0"/>
+    <origin xyz="0 -0.103 0" rpy="${PI/2} 0 0"/>
+  </joint>
+  <link name="servo5">
+    <visual>
+      <origin xyz="0.0 0.0 ${-servo_length/2}" rpy="0.0 0.0 0.0"/>
+      <geometry>
+        <cylinder radius="${servo_radius}" length="${servo_length}"/>
+      </geometry>
+      <material name="black"/>
+    </visual>
+    <collision>
+      <origin xyz="0.0 0.0 ${-servo_length/2}" rpy="0.0 0.0 0.0"/>
+      <geometry>
+        <cylinder radius="${servo_radius}" length="${servo_length}"/>
+      </geometry>
+      <material name="black"/>
+    </collision>
+    <xacro:cylinder mass="2" radius="${servo_radius}" height="${servo_length}"
+            xyz="0.0 0.0 ${-servo_length/2}" rpy="0.0 0.0 0.0"/>
+  </link>
+  <joint name="joint5" type="revolute">
+    <parent link="servo4"/>
+    <child link="servo5"/>
+    <axis xyz="0 0 1"/>
+    <limit lower="0" upper="${PI}" velocity="50.0" effort="1000.0"/>
+    <origin xyz="${servo_length} 0 0" rpy="${PI/2} 0 ${PI/2}"/>
+  </joint>
+  <link name="arm2">
+    <visual>
+      <origin xyz="-0.03 0.0 0.0" rpy="0.0 0.0 0.0"/>
+      <geometry>
+        <box size="0.06 0.02 0.001"/>
+      </geometry>
+      <material name="grey"/>
+    </visual>
+    <collision>
+      <origin xyz="-0.03 0.0 0.0" rpy="0.0 0.0 0.0"/>
+      <geometry>
+        <box size="${a4} 0.02 0.001"/>
+      </geometry>
+      <material name="grey"/>
+    </collision>
+    <xacro:box mass="0.2" length="0.06" width="0.001" height="0.02"
+          xyz="-0.03 0.0 0.0" rpy="0.0 0.0 0.0"/>
+  </link>
+  <joint name="arm2_joint" type="fixed">
+    <parent link="servo5"/>
+    <child link="arm2"/>
+    <origin xyz="0.06 0.0 0.0" rpy="${-PI/2} 0.0 0.0"/>
+  </joint>
+  <link name="servo6">
+    <visual>
+      <origin xyz="0.0 0.0 -0.03" rpy="0.0 0.0 0.0"/>
+      <geometry>
+        <cylinder radius="${servo_radius}" length="${servo_length}"/>
+      </geometry>
+      <material name="black"/>
+    </visual>
+    <collision>
+      <origin xyz="0.0 0.0 -0.03" rpy="0.0 0.0 0.0"/>
+      <geometry>
+        <cylinder radius="${servo_radius}" length="${servo_length}"/>
+      </geometry>
+      <material name="black"/>
+    </collision>
+    <xacro:cylinder mass="2" radius="${servo_radius}" height="${servo_length}"
+            xyz="0.0 0.0 -0.03" rpy="0.0 0.0 0.0"/>
+  </link>
+  <joint name="joint6" type="revolute">
+    <parent link="arm2"/>
+    <child link="servo6"/>
+    <axis xyz="0 0 1"/>
+    <limit lower="0" upper="${PI}" velocity="50.0" effort="1000.0"/>
+    <origin xyz="0.06 0 0" rpy="0 ${-3*PI/2} 0"/>
+  </joint>
+  <link name="gripper_support">
+    <visual>
+      <origin xyz="0.0 0.0 -0.03" rpy="0.0 ${PI/2} 0.0"/>
+      <geometry>
+        <box size="0.06 0.02 0.001"/>
+      </geometry>
+      <material name="grey"/>
+    </visual>
+    <collision>
+      <origin xyz="0.0 0.0 -0.03" rpy="0.0 ${PI/2} 0.0"/>
+      <geometry>
+        <box size="${a4} 0.02 0.001"/>
+      </geometry>
+      <material name="grey"/>
+    </collision>
+    <xacro:box mass="0.2" length="0.06" width="0.001" height="0.02"
+          xyz="0.0 0.0 -0.03" rpy="0.0 ${PI/2} 0.0"/>
+  </link>
+  <joint name="gripper_joint" type="fixed">
+    <parent link="servo6"/>
+    <child link="gripper_support"/>
+    <origin xyz="0.0 0.0 0.03" rpy="0.0 0.0 0.0"/>
+  </joint>
+  <link name="gripper_right">
+    <visual>
+        <origin rpy="0 0 0" xyz="-0.06 0.0 0.0"/>
+        <geometry>
+            <mesh filename="package://chessbot_description/meshes/left_finger.STL" scale="0.001 0.001 0.001"/>
+        </geometry>
+    </visual>
+    <collision>
+      <origin rpy="0 0 0" xyz="-0.06 0.0 0.0"/>
+        <geometry>
+            <mesh filename="package://chessbot_description/meshes/left_finger.STL" scale="0.001 0.001 0.001"/>
+        </geometry>
+    </collision>
+    <xacro:box mass="0.1" length="0.06" width="0.02" height="0.001"
+          rpy="0 0 0" xyz="-0.06 0.0 0.0"/>
+</link>
+<joint name ="joint7" type="revolute">
+  <parent link="gripper_support"/>
+  <child link = "gripper_right"/>
+  <origin xyz="0.0 -0.01 0.0" rpy="0.0 ${PI/2} 0.0"/>
+  <axis xyz="0 0 1"/>
+  <limit lower="0.0" upper="${7*PI/36}"
+         effort="1000" velocity="10"/>
+</joint>
+  <link name="gripper_left">
+    <visual>
+        <origin rpy="0 0 0" xyz="-0.06 0.0 0.0"/>
+        <geometry>
+            <mesh filename="package://chessbot_description/meshes/right_finger.STL" scale="0.001 0.001 0.001"/>
+        </geometry>
+    </visual>
+    <collision>
+      <origin rpy="0 0 0" xyz="-0.06 0.0 0.0"/>
+        <geometry>
+            <mesh filename="package://chessbot_description/meshes/right_finger.STL" scale="0.001 0.001 0.001"/>
+        </geometry>
+    </collision>
+    <xacro:box mass="0.1" length="0.06" width="0.02" height="0.001"
+          rpy="0 0 0" xyz="-0.06 0.0 0.0"/>
+</link>
+<joint name ="joint8" type="revolute">
+  <parent link="gripper_support"/>
+  <child link = "gripper_left"/>
+  <origin xyz="0.0 0.0 0.0" rpy="0.0 ${PI/2} 0.0"/>
+  <axis xyz="0 0 1"/>
+  <limit lower="${-7*PI/36}" upper="0.0"
+         effort="1000" velocity="10"/>
+         <mimic joint="joint7" multiplier="-1"/>
+</joint>
+<joint name="joint8_mimic" type="fixed">
+  <parent link="world" />
+  <child link="random" />
+</joint>
+<link name="random"/>
+    <xacro:arm_default_transmission joint_number="1"></xacro:arm_default_transmission>
+    <xacro:arm_default_transmission joint_number="2"></xacro:arm_default_transmission>
+    <xacro:arm_default_transmission joint_number="3"></xacro:arm_default_transmission>
+    <xacro:arm_default_transmission joint_number="4"></xacro:arm_default_transmission>
+    <xacro:arm_default_transmission joint_number="5"></xacro:arm_default_transmission>
+    <xacro:arm_default_transmission joint_number="6"></xacro:arm_default_transmission>
+    <xacro:arm_default_transmission joint_number="7"></xacro:arm_default_transmission>
+    <xacro:arm_default_transmission joint_number="8"></xacro:arm_default_transmission>
 </robot>

File: src/chessbot_description/urdf/arm_gazebo.urdf.xacro (robot description, xacro)
@@ -4,29 +4,32 @@
         <material>Gazebo/White</material>
     </gazebo>
-    <gazebo reference="link3">
+    <gazebo reference="servo1">
         <material>Gazebo/White</material>
     </gazebo>
-    <gazebo reference="link7">
-        <material>Gazebo/White</material>
-    </gazebo>
-    <gazebo reference="tool_tip">
-        <material>Gazebo/Yellow</material>
-    </gazebo>
-    <gazebo reference="link1">
+    <gazebo reference="servo2">
         <material>Gazebo/Black</material>
     </gazebo>
-    <gazebo reference="link2">
+    <gazebo reference="servo3">
         <material>Gazebo/Black</material>
     </gazebo>
-    <gazebo reference="link4">
+    <gazebo reference="servo4">
         <material>Gazebo/Black</material>
     </gazebo>
-    <gazebo reference="link5">
+    <gazebo reference="servo5">
         <material>Gazebo/Black</material>
     </gazebo>
-    <gazebo reference="link6">
+    <gazebo reference="servo6">
         <material>Gazebo/Black</material>
     </gazebo>
-    <gazebo reference="link8">
+    <gazebo reference="servo7">
+        <material>Gazebo/Black</material>
+    </gazebo>
+    <gazebo reference="servo8">
+        <material>Gazebo/Black</material>
+    </gazebo>
+    <gazebo reference="arm1">
+        <material>Gazebo/Black</material>
+    </gazebo>
+    <gazebo reference="arm2">
         <material>Gazebo/Black</material>
     </gazebo>
@@ -35,6 +38,6 @@
           <robot_param>robot_description</robot_param>
           <robot_param_node>robot_state_publisher</robot_param_node>
-          <parameters>$(find arm_controller)/config/robotarm_controllers.yaml</parameters>
+          <parameters>$(find chessbot_controller)/config/arm_controllers.yaml</parameters>
         </plugin>
-      </gazebo>
+    </gazebo>
 </robot>

File: src/chessbot_description/urdf/arm_ros2_control.urdf.xacro (robot description, xacro)
@@ -2,16 +2,8 @@
 <robot xmlns:xacro="http://www.ros.org/wiki/xacro">
     <ros2_control name="RobotSystem" type="system">
-        <xacro:if value="$(arg is_sim)">
-            <hardware>
-                <plugin>gazebo_ros2_control/GazeboSystem</plugin>
-            </hardware>
-        </xacro:if>
-        <xacro:unless value="$(arg is_sim)">
-            <hardware>
-                <plugin>arm_controller/RobotArmInterface</plugin>
-                <param name="port">/dev/ttyUSB0</param>
-            </hardware>
-        </xacro:unless>
-        <joint name="joint_1">
+        <hardware>
+            <plugin>gazebo_ros2_control/GazeboSystem</plugin>
+        </hardware>
+        <joint name="joint1">
             <command_interface name="position">
             <param name="min">0</param>
@@ -20,5 +12,5 @@
             <state_interface name="position"/>
         </joint>
-        <joint name="joint_2">
+        <joint name="joint2">
             <command_interface name="position">
             <param name="min">0</param>
@@ -27,5 +19,5 @@
             <state_interface name="position"/>
         </joint>
-        <joint name="joint_3">
+        <joint name="joint3">
             <command_interface name="position">
             <param name="min">0</param>
@@ -34,5 +26,5 @@
             <state_interface name="position"/>
         </joint>
-        <joint name="joint_4">
+        <joint name="joint4">
             <command_interface name="position">
             <param name="min">0</param>
@@ -41,5 +33,5 @@
             <state_interface name="position"/>
         </joint>
-        <joint name="joint_5">
+        <joint name="joint5">
             <command_interface name="position">
             <param name="min">0</param>
@@ -48,5 +40,5 @@
             <state_interface name="position"/>
         </joint>
-        <joint name="joint_6">
+        <joint name="joint6">
             <command_interface name="position">
             <param name="min">0</param>
@@ -55,4 +47,16 @@
             <state_interface name="position"/>
         </joint>
+        <joint name="joint7">
+            <command_interface name="position"/>
+            <state_interface name="position"/>
+            <limit lower="0" upper="${7*PI/36}" effort="1000" velocity="10"/>
+        </joint>
+        <joint name="joint8">
+            <param name="mimic">joint7</param>
+            <param name="multiplier">-1</param>
+            <command_interface name="position"/>
+            <state_interface name="position"/>
+            <limit lower="${-7*PI/36}" upper="0" effort="1000" velocity="10"/>
+        /</joint>
     </ros2_control>
 </robot>

File: src/chessbot_description/urdf/main.urdf.xacro (robot description, xacro)
@@ -4,5 +4,5 @@
     <xacro:include filename="arm_inertia.urdf.xacro"/>
     <xacro:include filename="arm_core.urdf.xacro"/>
-    <!-- <xacro:include filename="arm_gazebo.urdf.xacro"/> -->
-    <!-- <xacro:include filename="arm_ros2_control.urdf.xacro"/> -->
+    <xacro:include filename="arm_gazebo.urdf.xacro"/>
+    <xacro:include filename="arm_ros2_control.urdf.xacro"/>
 </robot>
