Commit message: fixed couple of issues

File: src/chessbot_description/urdf/arm_ros2_control.urdf.xacro (robot description, xacro)
@@ -2,7 +2,22 @@
 <robot xmlns:xacro="http://www.ros.org/wiki/xacro">
     <ros2_control name="RobotSystem" type="system">
-        <hardware>
-            <plugin>gazebo_ros2_control/GazeboSystem</plugin>
-        </hardware>
+        <xacro:if value="$(arg is_sim)">
+            <hardware>
+                <plugin>gazebo_ros2_control/GazeboSystem</plugin>
+            </hardware>
+            <joint name="joint8">
+                <param name="mimic">joint7</param>
+                <param name="multiplier">-1</param>
+                <command_interface name="position"/>
+                <state_interface name="position"/>
+                <limit lower="${-7*PI/36}" upper="0" effort="1000" velocity="10"/>
+            </joint>
+        </xacro:if>
+        <xacro:unless value="$(arg is_sim)">
+            <hardware>
+                <plugin>arm_controller/RobotArmInterface</plugin>
+                <param name="port">/dev/ttyUSB0</param>
+            </hardware>
+        </xacro:unless>
         <joint name="joint1">
             <command_interface name="position">
@@ -52,11 +67,4 @@
             <limit lower="0" upper="${7*PI/36}" effort="1000" velocity="10"/>
         </joint>
-        <joint name="joint8">
-            <param name="mimic">joint7</param>
-            <param name="multiplier">-1</param>
-            <command_interface name="position"/>
-            <state_interface name="position"/>
-            <limit lower="${-7*PI/36}" upper="0" effort="1000" velocity="10"/>
-        /</joint>
     </ros2_control>
 </robot>
